File: mysterium-pcb.kicad_pcb (KiCad board)
At the start: 2 copper layers, 347.7 x 146.6 mm, 224 parts, among them J1 AVR-ISP-6, SW1 KEYSW, SW10 KEYSW, SW11 KEYSW, SW12 KEYSW, SW13 KEYSW, SW14 KEYSW, SW15 KEYSW, SW16 KEYSW, SW17 KEYSW, SW18 KEYSW, SW19 KEYSW, SW2 KEYSW, SW20 KEYSW, SW21 KEYSW, SW22 KEYSW, SW23 KEYSW, SW24 KEYSW, SW25 KEYSW, SW26 KEYSW, SW27 KEYSW, SW28 KEYSW, SW29 KEYSW, SW3 KEYSW, SW30 KEYSW, SW31 KEYSW, SW32 KEYSW, SW33 KEYSW, SW34 KEYSW, SW35 KEYSW, SW36 KEYSW, SW37 KEYSW, SW38 KEYSW, SW39 KEYSW, SW4 KEYSW, SW40 KEYSW, SW41 KEYSW, SW42 KEYSW, SW43 KEYSW, SW44 KEYSW, SW45 KEYSW, SW46 KEYSW, SW47 KEYSW, SW48 KEYSW, SW49 KEYSW, SW5 KEYSW, SW50 KEYSW, SW51 KEYSW, SW52 KEYSW, SW53 KEYSW, SW54 KEYSW, SW55 KEYSW, SW56 KEYSW, SW57 KEYSW, SW58 KEYSW, SW59 KEYSW, SW6 KEYSW, SW60 KEYSW, SW61 KEYSW, SW62 KEYSW, SW63 KEYSW, SW64 KEYSW, SW65 KEYSW, SW66 KEYSW, SW67 KEYSW, SW68 KEYSW, SW69 KEYSW, SW7 KEYSW, SW70 KEYSW, SW71 KEYSW, SW72 KEYSW, SW73 KEYSW, SW74 KEYSW, SW75 KEYSW, SW76 KEYSW, SW77 KEYSW, SW78 KEYSW, SW79 KEYSW, SW8 KEYSW, SW80 KEYSW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

Commit message: Updated Gerbers
Parts:
- moved USB1 2.54 mm to (51.4, 57.8)
- moved BOOT1 2.54 mm to (60.9, 68.9)
- moved RESET1 2.54 mm to (48.2, 68.9)
Routing:
- net MOSI: track 296.6 -> 282.2 mm
- net GND: track 24.4 -> 18.3 mm
- net Net-(R2-Pad2): track 259.6 -> 263.2 mm
- net Net-(D77-Pad2): track 147.9 -> 144.4 mm
- net Net-(D64-Pad2): track 122.5 -> 119.0 mm
- net Net-(D34-Pad2): track 84.2 -> 80.7 mm
- net Net-(D51-Pad2): track 113.1 -> 109.7 mm
- net Net-(D17-Pad2): track 70.3 -> 66.9 mm
- net reset: track 312.7 -> 315.3 mm
- net Net-(D88-Pad1): track 354.9 -> 357.4 mm
- net boot: track 327.3 -> 329.9 mm
- net Net-(D89-Pad1): track 313.7 -> 315.3 mm
- net Net-(R5-Pad1): track 251.7 -> 253.2 mm
