File: bottom/mysterium-bottom.kicad_pcb (KiCad board)
At the start: 2 copper layers, 347.7 x 146.6 mm, 22 parts

Commit message: Updated Gerbers
Parts:
- removed G***: LOGO, logos:TOPY 4MM MASK
- removed G***: LOGO, logos:TOPY 4MM COPPER
- removed G***: LOGO, logos:MYSTERIUM_LARGE_COPPER
Other:
- net class Default removed
- board text removed: "coseyfannitutti"
